Commit message: fix small bug

File: gripper_descriptions/assets/x_grippers/surge_hand/gripper.urdf (robot description, URDF)
Before this commit: robot gripper, 12 links, 11 joints
Joints:
- joint Middle_MCP_Joint: limit lower=0 upper=1774 effort=10 velocity=5 -> lower=0 upper=1.774 effort=10 velocity=5

File: gripper_descriptions/assets/x_grippers/surge_hand/gripper_spherical_dof.urdf (robot description, URDF)
Before this commit: robot gripper, 16 links, 15 joints
Joints:
- joint Middle_MCP_Joint: limit lower=0 upper=1774 effort=10 velocity=5 -> lower=0 upper=1.774 effort=10 velocity=5
